Commit message: GOIDA

File: install/roarm_description/share/roarm_description/urdf/roarm_m3/materials.xacro (robot description, xacro)
@@ -1,6 +1 @@
-<?xml version="1.0" ?>
-<robot name="roarm_m3" xmlns:xacro="http://www.ros.org/wiki/xacro" >
-<material name="silver">
-  <color rgba="0.700 0.700 0.700 1.000"/>
-</material>
-</robot>
+/home/v1/Desktop/Beizo/arm_ws/build/roarm_description/urdf/roarm_m3/materials.xacro

File: install/roarm_description/share/roarm_description/urdf/roarm_m3/roarm_m3.xacro (robot description, xacro)
@@ -1,226 +1 @@
-<?xml version="1.0" ?>
-<robot name="roarm_m3" xmlns:xacro="http://www.ros.org/wiki/xacro">
-<xacro:include filename="$(find roarm_description)/urdf/roarm_m3/materials.xacro" />
-<!-- <xacro:include filename="$(find roarm_description)/urdf/roarm_m3/roarm_m3.trans" />
-<xacro:include filename="$(find roarm_description)/urdf/roarm_m3/roarm_m3.gazebo" /> -->
-<link name="world"></link>
-<link name="base_link">
-  <inertial>
-    <origin xyz="-0.0068 0 -0.03" rpy="0 0 0" />
-    <mass value="0.2562183" />
-    <inertia ixx="0.00029211" ixy="0" ixz="0" iyy="0.00035719" iyz="0" izz="0.000349421" />
-  </inertial>
-  <visual>
-    <origin xyz="0 0 0" rpy="0 0 0"/>
-    <geometry>
-      <mesh filename="file://$(find roarm_description)/meshes/roarm_m3/base_link.stl" scale="0.001 0.001 0.001"/>
-    </geometry>
-    <material name="silver"/>
-  </visual>
-  <collision>
-    <origin xyz="0 0 0" rpy="0 0 0"/>
-    <geometry>
-      <mesh filename="file://$(find roarm_description)/meshes/roarm_m3/base_link.stl" scale="0.001 0.001 0.001"/>
-    </geometry>
-  </collision>
-</link>
-<link name="link1">
-  <inertial>
-    <origin xyz="0 0 0.037" rpy="0 0 0" />
-    <mass value="0.0729177" />
-    <inertia ixx="4.68465E-05" ixy="0" ixz="0" iyy="3.32107E-05" iyz="0" izz="5.01023E-05" />
-  </inertial>
-  <visual>
-    <origin xyz="-0.0 -0.0 -0.0" rpy="0 0 0"/>
-    <geometry>
-      <mesh filename="file://$(find roarm_description)/meshes/roarm_m3/link1.stl" scale="0.001 0.001 0.001"/>
-    </geometry>
-    <material name="silver"/>
-  </visual>
-  <collision>
-    <origin xyz="-0.0 -0.0 -0.0" rpy="0 0 0"/>
-    <geometry>
-      <mesh filename="file://$(find roarm_description)/meshes/roarm_m3/link1.stl" scale="0.001 0.001 0.001"/>
-    </geometry>
-  </collision>
-</link>
-<link name="link2">
-  <inertial>
-    <origin xyz="0.119 0.012247 -0.0001 " rpy="0 0 0"/>
-    <mass value="0.0703216" />
-    <inertia ixx="5.46501E-05" ixy="0" ixz="0" iyy="0.000423091" iyz="0" izz="0.000404557" />
-  </inertial>
-  <visual>
-    <origin xyz="0 0 0" rpy="0 0 0"/>
-    <geometry>
-      <mesh filename="file://$(find roarm_description)/meshes/roarm_m3/link2.stl" scale="0.001 0.001 0.001"/>
-    </geometry>
-    <material name="silver"/>
-  </visual>
-  <collision>
-    <origin xyz="0 0 0" rpy="0 0 0"/>
-    <geometry>
-      <mesh filename="file://$(find roarm_description)/meshes/roarm_m3/link2.stl" scale="0.001 0.001 0.001"/>
-    </geometry>
-  </collision>
-</link>
-<link name="link3">
-  <inertial>
-    <origin xyz="-0.0015 -0.0765 0.00505" rpy="0 0 0"/>
-    <mass value="0.021608"/>
-    <inertia ixx="6.37699E-05" iyy="3.67026E-06" izz="6.28965E-05" ixy="0.0" iyz="0" ixz="0"/>
-  </inertial>
-  <visual>
-    <origin xyz="0 0 0" rpy="0 0 0"/>
-    <geometry>
-      <mesh filename="file://$(find roarm_description)/meshes/roarm_m3/link3.stl" scale="0.001 0.001 0.001"/>
-    </geometry>
-    <material name="silver"/>
-  </visual>
-  <collision>
-    <origin xyz="0 0 0" rpy="0 0 0"/>
-    <geometry>
-      <mesh filename="file://$(find roarm_description)/meshes/roarm_m3/link3.stl" scale="0.001 0.001 0.001"/>
-    </geometry>
-  </collision>
-</link>
-<link name="link4">
-  <inertial>
-    <origin xyz="-0.0015 -0.022 -0.00075" rpy="0 0 0"/>
-    <mass value="0.0099933"/>
-    <inertia ixx="4.53979E-06" iyy="3.78103E-06" izz="5.60238E-06" ixy="-0.0" iyz="-0.0" ixz="0.0"/>
-  </inertial>
-  <visual>
-    <origin xyz="0 0 0" rpy="0 0 0"/>
-    <geometry>
-      <mesh filename="file://$(find roarm_description)/meshes/roarm_m3/link4.stl" scale="0.001 0.001 0.001"/>
-    </geometry>
-    <material name="silver"/>
-  </visual>
-  <collision>
-    <origin xyz="0 0 0" rpy="0 0 0"/>
-    <geometry>
-      <mesh filename="file://$(find roarm_description)/meshes/roarm_m3/link4.stl" scale="0.001 0.001 0.001"/>
-    </geometry>
-  </collision>
-</link>
-<link name="link5">
-  <inertial>
-    <origin xyz="-0.0078 0 0.0595" rpy="0 0 0"/>
-    <mass value="0.0153928"/>
-    <inertia ixx="2.02869E-05" iyy="2.14427E-05" izz="4.39495E-06" ixy="-0.0" iyz="0" ixz="0"/>
-  </inertial>
-  <visual>
-    <origin xyz="0 0 0" rpy="0 0 0"/>
-    <geometry>
-      <mesh filename="file://$(find roarm_description)/meshes/roarm_m3/link5.stl" scale="0.001 0.001 0.001"/>
-    </geometry>
-    <material name="silver"/>
-  </visual>
-  <collision>
-    <origin xyz="0 0 0" rpy="0 0 0"/>
-    <geometry>
-      <mesh filename="file://$(find roarm_description)/meshes/roarm_m3/link5.stl" scale="0.001 0.001 0.001"/>
-    </geometry>
-  </collision>
-</link>
-<link name="gripper_link">
-  <inertial>
-    <origin xyz="0.027 0.0027 -0.018935" rpy="0 0 0"/>
-    <mass value="0.0028708" />
-    <inertia ixx="5.23216E-07" ixy="0" ixz="0" iyy="1.82071E-06" iyz="0" izz="1.60231E-06" />
-  </inertial>
-  <visual>
-    <origin xyz="0 0 0" rpy="0 0 0"/>
-    <geometry>
-      <mesh filename="file://$(find roarm_description)/meshes/roarm_m3/gripper_link.stl" scale="0.001 0.001 0.001"/>
-    </geometry>
-    <material name="silver"/>
-  </visual>
-  <collision>
-    <origin xyz="0 0 0" rpy="0 0 0"/>
-    <geometry>
-      <mesh filename="file://$(find roarm_description)/meshes/roarm_m3/gripper_link.stl" scale="0.001 0.001 0.001"/>
-    </geometry>
-  </collision>
-</link>
-<link name="hand_tcp"></link>
-<joint name="world_to_base_link" type="fixed">
-  <origin xyz="-0.12 0.0 0.04" rpy="0 0 0"/>
-  <parent link="world"/>
-  <child link="base_link"/>
-  <axis xyz="0.0 0.0 1.0"/>
-</joint>
-<joint name="base_link_to_link1" type="revolute">
-  <origin xyz="0.0 0.0 0.0" rpy="0 0 0"/>
-  <parent link="base_link"/>
-  <child link="link1"/>
-  <axis xyz="0.0 0.0 1.0"/>
-  <limit
-    lower="-3.1416"
-    upper="3.1416"
-    effort="1"
-    velocity="1" />
-</joint>
-<joint name="link1_to_link2" type="revolute">
-  <origin xyz="0.0 0.0 0.051959" rpy="-1.5708 -1.5708 0"/>
-  <parent link="link1"/>
-  <child link="link2"/>
-  <axis xyz="-0.0 0 1.0"/>
-  <limit
-    lower="-1.5708"
-    upper="1.5708"
-    effort="1"
-    velocity="1" />
-</joint>
-<joint name="link2_to_link3" type="revolute">
-  <origin xyz="0.236815 0.030002 0" rpy="0 0 1.5708"/>
-  <parent link="link2"/>
-  <child link="link3"/>
-  <axis xyz="0.0 0.0 1.0"/>
-  <limit
-    lower="-1"
-    upper="2.95"
-    effort="1"
-    velocity="1" />
-</joint>
-<joint name="link3_to_link4" type="revolute">
-  <origin xyz="0.0 -0.144586 0" rpy="0 0 0"/>
-  <parent link="link3"/>
-  <child link="link4"/>
-  <axis xyz="0.0 0.0 1.0"/>
-  <limit
-    lower="-1.5708"
-    upper="1.5708"
-    effort="1"
-    velocity="1" />
-</joint>
-<joint name="link4_to_link5" type="revolute">
-  <origin xyz="0.015147 -0.053653 0" rpy="1.5708 1.5708 0"/>
-  <parent link="link4"/>
-  <child link="link5"/>
-  <axis xyz="0.0 0.0 1.0"/>
-  <limit
-    lower="-3.1416"
-    upper="3.1416"
-    effort="1"
-    velocity="1" />
-</joint>
-<joint name="link5_to_gripper_link" type="revolute">
-  <origin xyz="0.00 0.018821 0.052035" rpy="-1.5708 -1.5708 0"/>
-  <parent link="link5"/>
-  <child link="gripper_link"/>
-  <axis xyz="0.0 -0.0 1.0"/>
-  <limit
-    lower="0"
-    upper="1.5"
-    effort="1"
-    velocity="1" />
-</joint>
-<joint name="link5_to_hand_tcp" type="fixed">
-  <origin xyz="0 0 0.115428" rpy="1.5708 -1.5708 0"/>
-  <parent link="link5"/>
-  <child link="hand_tcp"/>
-  <axis xyz="0 0 0"/>
-</joint>
-</robot>
+/home/v1/Desktop/Beizo/arm_ws/build/roarm_description/urdf/roarm_m3/roarm_m3.xacro

File: install/roarm_description/share/roarm_description/urdf/roarm_m3_description.xacro (robot description, xacro)
@@ -1,4 +1 @@
-<?xml version="1.0"?>
-<robot xmlns:xacro="http://www.ros.org/wiki/xacro" name="roarm_m3">
-    <xacro:include filename="$(find roarm_description)/urdf/roarm_m3/roarm_m3.xacro" />
-</robot>
+/home/v1/Desktop/Beizo/arm_ws/build/roarm_description/urdf/roarm_m3_description.xacro

File: install/roarm_description/share/roarm_description/urdf/roarm_m3_moveit.xacro (robot description, xacro)
@@ -1,4 +1 @@
-<?xml version="1.0"?>
-<robot xmlns:xacro="http://www.ros.org/wiki/xacro" name="roarm_m3">
-    <xacro:include filename="$(find roarm_description)/urdf/roarm_m3/roarm_m3.xacro" />
-</robot>
+/home/v1/Desktop/Beizo/arm_ws/build/roarm_description/urdf/roarm_m3_moveit.xacro

File: install/roarm_moveit_config/share/roarm_moveit_config/config/roarm_m3.ros2_control.xacro (robot description, xacro)
@@ -1,54 +1 @@
-<?xml version="1.0"?>
-<robot xmlns:xacro="http://www.ros.org/wiki/xacro">
-    <xacro:macro name="roarm_m3_ros2_control" params="name initial_positions_file">
-        <xacro:property name="initial_positions" value="${xacro.load_yaml(initial_positions_file)['initial_positions']}"/>
-        <ros2_control name="${name}" type="system">
-            <hardware>
-                <!-- By default, set up controllers for simulation. This won't work on real hardware -->
-                <plugin>mock_components/GenericSystem</plugin>
-            </hardware>
-            <joint name="base_link_to_link1">
-                <command_interface name="position"/>
-                <state_interface name="position">
-                  <param name="initial_value">${initial_positions['base_link_to_link1']}</param>
-                </state_interface>
-                <state_interface name="velocity"/>
-            </joint>
-            <joint name="link1_to_link2">
-                <command_interface name="position"/>
-                <state_interface name="position">
-                  <param name="initial_value">${initial_positions['link1_to_link2']}</param>
-                </state_interface>
-                <state_interface name="velocity"/>
-            </joint>
-            <joint name="link2_to_link3">
-                <command_interface name="position"/>
-                <state_interface name="position">
-                  <param name="initial_value">${initial_positions['link2_to_link3']}</param>
-                </state_interface>
-                <state_interface name="velocity"/>
-            </joint>
-            <joint name="link3_to_link4">
-                <command_interface name="position"/>
-                <state_interface name="position">
-                  <param name="initial_value">${initial_positions['link3_to_link4']}</param>
-                </state_interface>
-                <state_interface name="velocity"/>
-            </joint>
-            <joint name="link4_to_link5">
-                <command_interface name="position"/>
-                <state_interface name="position">
-                  <param name="initial_value">${initial_positions['link4_to_link5']}</param>
-                </state_interface>
-                <state_interface name="velocity"/>
-            </joint>
-            <joint name="link5_to_gripper_link">
-                <command_interface name="position"/>
-                <state_interface name="position">
-                  <param name="initial_value">${initial_positions['link5_to_gripper_link']}</param>
-                </state_interface>
-                <state_interface name="velocity"/>
-            </joint>
-        </ros2_control>
-    </xacro:macro>
-</robot>
+/home/v1/Desktop/Beizo/arm_ws/src/roarm_moveit_config/config/roarm_m3.ros2_control.xacro

File: install/roarm_moveit_config/share/roarm_moveit_config/config/roarm_m3.urdf.xacro (robot description, xacro)
@@ -1,7 +1 @@
-<?xml version="1.0"?>
-<robot xmlns:xacro="http://www.ros.org/wiki/xacro" name="roarm_m3">
-    <xacro:arg name="initial_positions_file" default="initial_positions.yaml" />
-    <xacro:include filename="$(find roarm_description)/urdf/roarm_m3/roarm_m3.xacro" />
-    <xacro:include filename="roarm_m3.ros2_control.xacro" />
-    <xacro:roarm_m3_ros2_control name="FakeSystem" initial_positions_file="$(arg initial_positions_file)"/>
-</robot>
+/home/v1/Desktop/Beizo/arm_ws/src/roarm_moveit_config/config/roarm_m3.urdf.xacro

File: src/roarm_description/urdf/roarm_m3/roarm_m3.xacro (robot description, xacro)
@@ -214,5 +214,5 @@
   <limit
     lower="0"
-    upper="1.5"
+    upper="3.15"
     effort="1"
     velocity="1" />
